Commit message: Got livox working on turtlebot, fixed frame transforms in plugin

File: livox_laser_simulation/urdf/livox_avia.xacro (robot description, xacro)
@@ -25,35 +25,35 @@
         <!-- This ray plgin is only for visualization. -->
         <plugin name="gazebo_ros_laser_controller" filename="liblivox_laser_simulation.so">
-			<ray>
-			  <scan>
-				<horizontal>
-				<samples>100</samples>
-				<resolution>1</resolution>
-				<min_angle>${-horizontal_fov/360*M_PI}</min_angle>
-				<max_angle>${horizontal_fov/360*M_PI}</max_angle>
-				</horizontal>
-				<vertical>
-				<samples>50</samples>
-				<resolution>1</resolution>
-				<min_angle>${-vertical_fov/360*M_PI}</min_angle>
-				<max_angle>${vertical_fov/360*M_PI}</max_angle>
-				</vertical>
-			  </scan>
-			  <range>
-				<min>${laser_min_range}</min>
-				<max>${laser_max_range}</max>
-				<resolution>${resolution}</resolution>
-			  </range>
-			  <noise>
-				<type>gaussian</type>
-				<mean>${noise_mean}</mean>
-				<stddev>${noise_stddev}</stddev>
-			  </noise>
-			</ray>
+          <ray>
+            <scan>
+              <horizontal>
+              <samples>100</samples>
+              <resolution>1</resolution>
+              <min_angle>${-horizontal_fov/360*M_PI}</min_angle>
+              <max_angle>${horizontal_fov/360*M_PI}</max_angle>
+              </horizontal>
+              <vertical>
+              <samples>50</samples>
+              <resolution>1</resolution>
+              <min_angle>${-vertical_fov/360*M_PI}</min_angle>
+              <max_angle>${vertical_fov/360*M_PI}</max_angle>
+              </vertical>
+            </scan>
+            <range>
+              <min>${laser_min_range}</min>
+              <max>${laser_max_range}</max>
+              <resolution>${resolution}</resolution>
+            </range>
+            <noise>
+              <type>gaussian</type>
+              <mean>${noise_mean}</mean>
+              <stddev>${noise_stddev}</stddev>
+            </noise>
+          </ray>
           <visualize>${visualize}</visualize>
-		  <samples>${samples}</samples>
-		  <downsample>${downsample}</downsample>
-		  <csv_file_name>package://livox_laser_simulation/scan_mode/avia.csv</csv_file_name>
-		  <ros_topic>${ros_topic}</ros_topic>
+          <samples>${samples}</samples>
+          <downsample>${downsample}</downsample>
+          <csv_file_name>package://livox_laser_simulation/scan_mode/avia.csv</csv_file_name>
+          <ros_topic>${ros_topic}</ros_topic>
         </plugin>
       </sensor>
@@ -88,5 +88,5 @@
     <xacro:Livox_Mid_gazebo_sensor name="${name}" visualize="${visualize}"/>
   </xacro:macro>
-    <xacro:Livox_AVIA name="livox"/>
+  <xacro:Livox_AVIA name="livox"/>
   <xacro:include filename="$(find livox_laser_simulation)/urdf/standardrobots_oasis300.xacro"/>
   <xacro:link_oasis name="oasis"/>

File: livox_laser_simulation/urdf/standardrobots_oasis300.xacro (robot description, xacro)
@@ -26,37 +26,37 @@
 -->
 	<xacro:macro name="link_oasis" params="name:=oasis base_link:=oasis_300 world_link:=link">
-    <link name="link"/>
-    <!-- base_link -->
-    <link name="oasis_300">
-        <visual>
-			<origin xyz="0.00 0 0.05" rpy="0 0 0"/>
-            <geometry>
-				  <mesh filename="package://livox_laser_simulation/meshes/standardrobots.STL"/>
-            </geometry>
-        </visual>
-        <collision>
-			<origin xyz="0.00 0 0.05" rpy="0 0 0"/>
-            <geometry>
-				  <mesh filename="package://livox_laser_simulation/meshes/standardrobots.STL"/>
-            </geometry>
-        </collision>
-        <xacro:inertial_matrix mass="1"/>
-		<kinematic>1</kinematic>
-		<gravity>9.8</gravity>
-    </link>
-    <gazebo reference="oasis_300">
-        <material>Gazebo/White</material>
-    </gazebo>
-	<joint name="fixed" type="fixed">
-		<parent link="${world_link}"/>
-		<child link="${base_link}"/>
-		<origin xyz="0.0 0 0.05" rpy="0 0 ${M_PI/2}" />
-	</joint>
-	<joint name="livox_base_joint" type="fixed">
-        <parent link="${base_link}"/>
-        <child link="livox_base"/>
-        <origin rpy="0 0 1.5707"
-                xyz="0.0 0.4 0.3057"/>
-    </joint>
+        <link name="link"/>
+        <!-- base_link -->
+        <link name="oasis_300">
+            <visual>
+                <origin xyz="0.00 0 0.05" rpy="0 0 0"/>
+                <geometry>
+                    <mesh filename="package://livox_laser_simulation/meshes/standardrobots.STL"/>
+                </geometry>
+            </visual>
+            <collision>
+                <origin xyz="0.00 0 0.05" rpy="0 0 0"/>
+                <geometry>
+                    <mesh filename="package://livox_laser_simulation/meshes/standardrobots.STL"/>
+                </geometry>
+            </collision>
+            <xacro:inertial_matrix mass="1"/>
+            <kinematic>1</kinematic>
+            <gravity>9.8</gravity>
+        </link>
+        <gazebo reference="oasis_300">
+            <material>Gazebo/White</material>
+        </gazebo>
+        <joint name="fixed" type="fixed">
+            <parent link="${world_link}"/>
+            <child link="${base_link}"/>
+            <origin xyz="0.0 0 0.05" rpy="0 0 ${M_PI/2}" />
+        </joint>
+        <joint name="livox_base_joint" type="fixed">
+            <parent link="${base_link}"/>
+            <child link="livox_base"/>
+            <origin rpy="0 0 1.5707"
+                    xyz="0.0 0.4 0.3057"/>
+        </joint>
     </xacro:macro>
 </robot>

File: mmslam/urdf/turtlebot.gazebo.xacro (robot description, xacro)
@@ -181,8 +181,3 @@
     <maxVel>0.1</maxVel>
   </gazebo>
-  <xacro:include filename="$(find velodyne_description)/urdf/VLP-16.urdf.xacro"/>
-  <xacro:VLP-16 parent="base_scan" name="velodyne" topic="/velodyne_points" organize_cloud="false" hz="20" samples="440" gpu="true">
-    <origin xyz="0 0 0.02" rpy="0 0 0" />
-    <!-- <origin xyz="-0.032 0 0.172" rpy="0 0 0"/> -->
-  </xacro:VLP-16>
 </robot>

File: mmslam/urdf/turtlebot.urdf.xacro (robot description, xacro)
@@ -164,3 +164,15 @@
     <origin xyz="-0.032 0 0.198" rpy="0 0 0"/>
   </joint>
+  <xacro:include filename="$(find velodyne_description)/urdf/VLP-16.urdf.xacro"/>
+  <xacro:VLP-16 parent="base_link" name="velodyne" topic="/velodyne_points" organize_cloud="false" hz="20" samples="440" gpu="true">
+    <!-- <origin xyz="0 0 0.02" rpy="0 0 0" /> -->
+    <origin xyz="-0.032 0 0.172" rpy="0 0 0"/>
+  </xacro:VLP-16>
+  <xacro:include filename="$(find mmslam)/urdf/livox.xacro"/>
+  <xacro:Livox_AVIA name="livox" visualize="true"/>
+  <joint name="livox_joint" type="fixed">
+    <parent link="base_link"/>
+    <child link="livox_base"/>
+    <origin xyz="-0.032 0 .198"/>
+  </joint>
 </robot>
