Commit message: Fixed extrinsic R matrix, removed livox from urdf

File: mmslam/urdf/turtlebot.urdf.xacro (robot description, xacro)
@@ -169,5 +169,5 @@
     <origin xyz="-0.032 0 0.172" rpy="0 0 0"/>
   </xacro:VLP-16>
-  <xacro:include filename="$(find mmslam)/urdf/livox.xacro"/>
+  <!-- <xacro:include filename="$(find mmslam)/urdf/livox.xacro"/>
   <xacro:Livox_AVIA name="livox" visualize="false"/>
   <joint name="livox_joint" type="fixed">
@@ -175,4 +175,4 @@
     <child link="livox_base"/>
     <origin xyz="-0.032 0 .198"/>
-  </joint>
+  </joint> -->
 </robot>

Commit message: Changing fast lio frames

File: mmslam/urdf/turtlebot.urdf.xacro (robot description, xacro)
@@ -162,5 +162,5 @@
     <parent link="base_link"/>
     <child link="base_camera"/>
-    <origin xyz="-0.032 0 0.198" rpy="0 0 0"/>
+    <origin xyz="-0.032 0 0.298" rpy="0 0 0"/>
   </joint>
   <xacro:include filename="$(find velodyne_description)/urdf/VLP-16.urdf.xacro"/>
